File: pwr.kicad_sch (KiCad schematic)
At the start: 41 parts, among them J2 XT90PW-M, J5 SAFETY, Q1 IRFP1405PBF, U1 AP1501_3.3, U2 AP1501_5, U3 AP1501_ADJ_7.5

Commit message: Added lambda connection, switching between PWM and 3.3v signal to drive mosfets.
Parts:
- added C29: 1000uF, Capacitor_THT:CP_Radial_D8.0mm_P3.50mm, symbol Device:C_Polarized
Connections:
- net +3.3V: now also C29.1
- net GND: now also C29.2
Other:
- moved on the sheet: C7
Changed lines of the file:
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@@
   (junction (at 31.75 53.34) (diameter 0) (color 0 0 0 0)
   )
-  (junction (at 264.16 53.34) (diameter 0) (color 0 0 0 0)
-  )
   (junction (at 228.6 73.66) (diameter 0) (color 0 0 0 0)
   )
   (junction (at 198.12 127) (diameter 0) (color 0 0 0 0)
   )
+  (junction (at 259.08 38.1) (diameter 0) (color 0 0 0 0)
+  )
   (junction (at 228.6 53.34) (diameter 0) (color 0 0 0 0)
   )
@@
   (junction (at 210.82 53.34) (diameter 0) (color 0 0 0 0)
   )
+  (junction (at 259.08 53.34) (diameter 0) (color 0 0 0 0)
+  )
   (junction (at 246.38 53.34) (diameter 0) (color 0 0 0 0)
   )
@@
   (junction (at 246.38 73.66) (diameter 0) (color 0 0 0 0)
   )
+  (junction (at 269.24 38.1) (diameter 0) (color 0 0 0 0)
+  )
   (junction (at 264.16 88.9) (diameter 0) (color 0 0 0 0)
   )
   (junction (at 107.95 31.75) (diameter 0) (color 0 0 0 0)
   )
-  (junction (at 264.16 38.1) (diameter 0) (color 0 0 0 0)
+  (junction (at 269.24 53.34) (diameter 0) (color 0 0 0 0)
   )
   (wire (pts (xy 242.57 38.1) (xy 246.38 38.1))
@@
     (stroke (width 0) (type default) (color 0 0 0 0))
   )
+  (wire (pts (xy 259.08 38.1) (xy 269.24 38.1))
+    (stroke (width 0) (type default) (color 0 0 0 0))
+  )
   (wire (pts (xy 264.16 88.9) (xy 275.59 88.9))
     (stroke (width 0) (type default) (color 0 0 0 0))
@@
     (stroke (width 0) (type default) (color 0 0 0 0))
   )
+  (wire (pts (xy 259.08 53.34) (xy 269.24 53.34))
+    (stroke (width 0) (type default) (color 0 0 0 0))
+  )
   (wire (pts (xy 175.26 96.52) (xy 175.26 106.68))
     (stroke (width 0) (type default) (color 0 0 0 0))
   )
-  (wire (pts (xy 264.16 53.34) (xy 246.38 53.34))
-    (stroke (width 0) (type default) (color 0 0 0 0))
-  )
   (wire (pts (xy 39.37 55.88) (xy 39.37 63.5))
     (stroke (width 0) (type default) (color 0 0 0 0))
@@
     (stroke (width 0) (type default) (color 0 0 0 0))
   )
-  (wire (pts (xy 264.16 48.26) (xy 264.16 53.34))
+  (wire (pts (xy 259.08 48.26) (xy 259.08 53.34))
     (stroke (width 0) (type default) (color 0 0 0 0))
   )
@@
     (stroke (width 0) (type default) (color 0 0 0 0))
   )
+  (wire (pts (xy 269.24 38.1) (xy 269.24 40.64))
+    (stroke (width 0) (type default) (color 0 0 0 0))
+  )
   (wire (pts (xy 264.16 127) (xy 246.38 127))
     (stroke (width 0) (type default) (color 0 0 0 0))
@@
     (stroke (width 0) (type default) (color 0 0 0 0))
   )
+  (wire (pts (xy 246.38 38.1) (xy 259.08 38.1))
+    (stroke (width 0) (type default) (color 0 0 0 0))
+  )
   (wire (pts (xy 228.6 73.66) (xy 223.52 73.66))
     (stroke (width 0) (type default) (color 0 0 0 0))
@@
     (stroke (width 0) (type default) (color 0 0 0 0))
   )
-  (wire (pts (xy 246.38 38.1) (xy 264.16 38.1))
-    (stroke (width 0) (type default) (color 0 0 0 0))
-  )
   (wire (pts (xy 246.38 83.82) (xy 246.38 88.9))
     (stroke (width 0) (type default) (color 0 0 0 0))
@@
     (stroke (width 0) (type default) (color 0 0 0 0))
   )
+  (wire (pts (xy 269.24 38.1) (xy 275.59 38.1))
+    (stroke (width 0) (type default) (color 0 0 0 0))
+  )
   (wire (pts (xy 246.38 91.44) (xy 254 91.44))
     (stroke (width 0) (type default) (color 0 0 0 0))
@@
     (stroke (width 0) (type default) (color 0 0 0 0))
   )
+  (wire (pts (xy 269.24 53.34) (xy 275.59 53.34))
+    (stroke (width 0) (type default) (color 0 0 0 0))
+  )
   (wire (pts (xy 182.88 29.21) (xy 182.88 33.02))
     (stroke (width 0) (type default) (color 0 0 0 0))
   )
+  (wire (pts (xy 269.24 48.26) (xy 269.24 53.34))
+    (stroke (width 0) (type default) (color 0 0 0 0))
+  )
   (wire (pts (xy 228.6 49.53) (xy 228.6 53.34))
     (stroke (width 0) (type default) (color 0 0 0 0))
@@
     (stroke (width 0) (type default) (color 0 0 0 0))
   )
-  (wire (pts (xy 264.16 38.1) (xy 275.59 38.1))
-    (stroke (width 0) (type default) (color 0 0 0 0))
-  )
   (wire (pts (xy 246.38 111.76) (xy 246.38 114.3))
     (stroke (width 0) (type default) (color 0 0 0 0))
@@
     (stroke (width 0) (type default) (color 0 0 0 0))
   )
-  (wire (pts (xy 264.16 38.1) (xy 264.16 40.64))
+  (wire (pts (xy 259.08 38.1) (xy 259.08 40.64))
     (stroke (width 0) (type default) (color 0 0 0 0))
   )
@@
     (stroke (width 0) (type default) (color 0 0 0 0))
   )
+  (wire (pts (xy 246.38 53.34) (xy 259.08 53.34))
+    (stroke (width 0) (type default) (color 0 0 0 0))
+  )
   (wire (pts (xy 118.11 52.07) (xy 118.11 41.91))
-    (stroke (width 0) (type default) (color 0 0 0 0))
-  )
-  (wire (pts (xy 264.16 53.34) (xy 275.59 53.34))
     (stroke (width 0) (type default) (color 0 0 0 0))
   )
@@
     (pin "4")
   )
-  (symbol (lib_id "power:+3.3V") (at 264.16 38.1 0) (unit 1)
-    (in_bom yes) (on_board yes) (fields_autoplaced)
-    (property "Reference" "#PWR0102" (id 0) (at 264.16 41.91 0)
-      (effects (font (size 1.27 1.27)) hide)
-    )
-    (property "Value" "+3.3V" (id 1) (at 264.16 33.02 0))
-    (property "Footprint" "" (id 2) (at 264.16 38.1 0)
-      (effects (font (size 1.27 1.27)) hide)
-    )
-    (property "Datasheet" "" (id 3) (at 264.16 38.1 0)
+  (symbol (lib_id "power:+3.3V") (at 269.24 38.1 0) (unit 1)
+    (in_bom yes) (on_board yes) (fields_autoplaced)
+    (property "Reference" "#PWR0102" (id 0) (at 269.24 41.91 0)
+      (effects (font (size 1.27 1.27)) hide)
+    )
+    (property "Value" "+3.3V" (id 1) (at 269.24 33.02 0))
+    (property "Footprint" "" (id 2) (at 269.24 38.1 0)
+      (effects (font (size 1.27 1.27)) hide)
+    )
+    (property "Datasheet" "" (id 3) (at 269.24 38.1 0)
       (effects (font (size 1.27 1.27)) hide)
     )
@@
   )
   (symbol (lib_id "Device:C_Polarized") (at 246.38 44.45 0) (unit 1)
-    (in_bom yes) (on_board yes) (fields_autoplaced)
-    (property "Reference" "C4" (id 0) (at 250.19 42.2909 0)
-      (effects (font (size 1.27 1.27)) (justify left))
-    )
-    (property "Value" "330uF" (id 1) (at 250.19 44.8309 0)
+    (in_bom yes) (on_board yes)
+    (property "Reference" "C4" (id 0) (at 247.65 49.53 0)
+      (effects (font (size 1.27 1.27)) (justify left))
+    )
+    (property "Value" "330uF" (id 1) (at 247.65 46.99 0)
       (effects (font (size 1.27 1.27)) (justify left))
     )
@@
     (pin "5")
   )
+  (symbol (lib_id "Device:C_Polarized") (at 269.24 44.45 0) (unit 1)
+    (in_bom yes) (on_board yes)
+    (property "Reference" "C29" (id 0) (at 270.51 49.53 0)
+      (effects (font (size 1.27 1.27)) (justify left))
+    )
+    (property "Value" "1000uF" (id 1) (at 270.51 46.99 0)
+      (effects (font (size 1.27 1.27)) (justify left))
+    )
+    (property "Footprint" "Capacitor_THT:CP_Radial_D8.0mm_P3.50mm" (id 2) (at 270.2052 48.26 0)
+      (effects (font (size 1.27 1.27)) hide)
+    )
+    (property "Datasheet" "~" (id 3) (at 269.24 44.45 0)
+      (effects (font (size 1.27 1.27)) hide)
+    )
+    (pin "1")
+    (pin "2")
+  )
   (symbol (lib_id "3557-2:3557-2") (at 82.55 36.83 90) (unit 1)
     (in_bom yes) (on_board yes)
@@
     (pin "4")
   )
-  (symbol (lib_id "Device:C") (at 264.16 44.45 0) (unit 1)
-    (in_bom yes) (on_board yes) (fields_autoplaced)
-    (property "Reference" "C7" (id 0) (at 267.97 43.1799 0)
-      (effects (font (size 1.27 1.27)) (justify left))
-    )
-    (property "Value" "0.1uF" (id 1) (at 267.97 45.7199 0)
-      (effects (font (size 1.27 1.27)) (justify left))
-    )
-    (property "Footprint" "Capacitor_SMD:C_0603_1608Metric" (id 2) (at 265.1252 48.26 0)
-      (effects (font (size 1.27 1.27)) hide)
-    )
-    (property "Datasheet" "~" (id 3) (at 264.16 44.45 0)
-      (effects (font (size 1.27 1.27)) hide)
-    )
+  (symbol (lib_id "Device:C") (at 259.08 44.45 0) (unit 1)
+    (in_bom yes) (on_board yes)
+    (property "Reference" "C7" (id 0) (at 260.35 49.53 0)
+      (effects (font (size 1.27 1.27)) (justify left))
+    )
+    (property "Value" "0.1uF" (id 1) (at 260.35 46.99 0)
+      (effects (font (size 1.27 1.27)) (justify left))
+    )
+    (property "Footprint" "Capacitor_SMD:C_0603_1608Metric" (id 2) (at 260.0452 48.26 0)
+      (effects (font (size 1.27 1.27)) hide)
+    )
+    (property "Datasheet" "~" (id 3) (at 259.08 44.45 0)
+      (effects (font (size 1.27 1.27)) hide)
+    )
