File: pwr.kicad_sch (KiCad schematic)
At the start: 42 parts, among them J2 XT90PW-M, J5 SAFETY, Q1 IRFP1405PBF, U1 AP1501_3.3, U2 AP1501_5, U3 AP1501_ADJ_7.5

Commit message: Added schematic descriptions
Other:
- note added: "Fuses"
- note added: "Main power connection for 16V LiPo"
- note added: "Power consumption safety measure section. It provides fuse holders for different parts of the circuit inlduing: - EMU Black (EMU) - Fuel injector (INJ) - Ignition coil (IGN) - Motor starter(STARTER) - 3.3V line (3.3V) - 5V line (5V) - 7.5V line (7.5V) - 16V line (16V)"
- note added: "Power section"
- note added: "This section includes various step-down voltage converters that include: 3.3V, 5V and 7.5V"
- note added: "This section uses a mosfet transistor to provide power to the circuit if its Gate is powered."
- note added: "Voltage converters"
- moved on the sheet: F1, F2, F3, F4, F5, F6, F7, F9

Commit message: Added 12V regulator for injector
Parts:
- added C31: 0.1uF, Capacitor_SMD:C_0603_1608Metric, symbol Device:C
- added C32: 0.22uF, Capacitor_SMD:C_0603_1608Metric, symbol Device:C
- added U11: LM340S-12/NOPB, lib:TO254P1524X483-4N, symbol LM340S-12_NOPB:LM340S-12/NOPB
- C29: footprint Capacitor_THT:CP_Radial_D8.0mm_P3.50mm -> Capacitor_THT:CP_Radial_D10.0mm_P7.50mm
Connections:
- net GND: now also C31.2, C32.2, U11.2 (GND), U11.4 (GND)
- net INJ: now also C32.1, U11.1 (IN)
- new net INJ_12V: C31.1, U11.3 (OUT)
Other:
- note added: "12V injector regulator"
