File: io.kicad_sch (KiCad schematic)
At the start: 39 parts, among them J10 RIGHT WHEEL SENS, J11 STARTER CON, J14 CAN, J15 3.3V OUT, J16 5V OUT, J17 7.5V OUT, J18 OIL CON, J19 IAT CON, J20 PRIM TRIGG CON, J21 SEC TRIGG CON, J22 EGT CON, J23 DATA LOGGER CON, J24 IGN CON, J25 INJ CON, J26 MAP, J27 CLT CON, J28 TPS CON, J29 WBO CON, J3 EMU_BLACK_A, J4 EMU_BLACK_B, J6 INJ_&_STARTER, J7 16V OUT, J8 SERVO, J9 LEFT WHEEL SENS, K1 FINDER-34.51 INJ, K2 FINDER-34.51 STARTER, K3 FINDER-34.51 INJ, Q2 IRFP1405PBF, Q3 IRFP1405PBF, Q4 IRFP1405PBF, U7 TXS0108EPWR

Commit message: Added schematic descriptions
Other:
- note added: "Connectors for 7.5V servomechanism and wheel HAL sensors"
- note added: "Driver buttons input Injector drive output"
- note added: "ECU Master EMU Black signal I/O"
- note added: "I/O section"
- note added: "Logic converter"
- note added: "Relays that allow converting 16V signals from driver buttons to 3.3V signals for RP2040 to read. One of th relays drive the enabling of the fuel injector"
- note added: "Sensors, Data Logger, CAN Bus, Power outputs"
- note added: "Servo / Wheel sensors"
- note added: "This chip allows to get signals from 5V sensors and drive MOSFET transistors on the RP2040 side"
- note added: "This connectors establish the connection between the board and the EMU Black computer including the supply of power to the computer, sensor readings, data logger and CAN Bus connections"
- note added: "Various connectors for external sensor connections, power line connections, CAN Bus I/O etc."
- moved on the sheet: C15, C16, J10, J25, J8, J9, K3, R14, S1, U7

Commit message: Added 12V regulator for injector
Connections:
- net INJ renamed INJ_12V
